Commit message: Integrating ros2_control with Gazebo to enable hardware interface and controller management.

File: my_bot/description/camera.xacro (robot description, xacro)
@@ -1,5 +1,5 @@
 <?xml version="1.0"?>
 <robot xmlns:xacro="http://www.ros.org/wiki/xacro">
-    <xacro:property name="pi" value="3.14159265359"/>
+    <xacro:property name="pi" value="3.141592653589793" unless="pi"/>
     <joint name="camera_joint" type="fixed">
         <parent link="chassis"/>

File: my_bot/description/depth_camera.xacro (robot description, xacro)
@@ -1,5 +1,5 @@
 <?xml version="1.0"?>
 <robot xmlns:xacro="http://www.ros.org/wiki/xacro">
-    <xacro:property name="pi" value="3.14159265359"/>
+    <!-- <xacro:property name="pi" value="3.14159265359"/> -->
     <joint name="depth_camera_joint" type="fixed">
         <parent link="chassis"/>

File: my_bot/description/robot.urdf.xacro (robot description, xacro)
@@ -4,5 +4,6 @@
     <!-- <link name="base_link"></link> -->
     <xacro:include filename="robot_core.xacro"/>
-    <xacro:include filename="gazebo_plugins.xacro"/>
+    <!-- <xacro:include filename="gazebo_control.xacro"/>  -->
+    <xacro:include filename="ros2_control.xacro"/>
     <xacro:include filename="lidar.xacro"/>
     <xacro:include filename="camera.xacro"/>

File: my_bot/description/robot_core.xacro (robot description, xacro)
@@ -2,5 +2,5 @@
 <robot xmlns:xacro="http://www.ros.org/wiki/xacro"  >
     <xacro:include filename="inertial_macros.xacro"/>
-    <xacro:property name="pi" value="3.14159265359"/>
+    <!-- <xacro:property name="pi" value="3.14159265359"/> -->
     <material name="white">
         <color rgba="1 1 1 1"/>

Commit message: Refactor launch files to support ROS 2 control configuration and improve simulation timing, and bug fix

File: my_bot/description/camera.xacro (robot description, xacro)
@@ -1,5 +1,4 @@
 <?xml version="1.0"?>
 <robot xmlns:xacro="http://www.ros.org/wiki/xacro">
-    <xacro:property name="pi" value="3.141592653589793" unless="pi"/>
     <joint name="camera_joint" type="fixed">
         <parent link="chassis"/>

File: my_bot/description/robot.urdf.xacro (robot description, xacro)
@@ -1,9 +1,17 @@
 <?xml version="1.0"?>
-<robot xmlns:xacro="http://www.ros.org/wiki/xacro"  name="robot">
-    <!-- Example link -->
-    <!-- <link name="base_link"></link> -->
+<robot xmlns:xacro="http://www.ros.org/wiki/xacro" name="robot">
+    <!-- Argument to switch between ros2_control and Gazebo control -->
+    <xacro:arg name="use_ros2_control" default="true"/>
+    <!-- Core robot body -->
     <xacro:include filename="robot_core.xacro"/>
-    <!-- <xacro:include filename="gazebo_control.xacro"/>  -->
-    <xacro:include filename="ros2_control.xacro"/>
+    <!-- ROS 2 Control -->
+    <xacro:if value="$(arg use_ros2_control)">
+        <xacro:include filename="ros2_control.xacro"/>
+    </xacro:if>
+    <!-- Gazebo control (if not using ros2_control) -->
+    <xacro:unless value="$(arg use_ros2_control)">
+        <xacro:include filename="gazebo_control.xacro"/>
+    </xacro:unless>
+    <!-- Sensors -->
     <xacro:include filename="lidar.xacro"/>
     <xacro:include filename="camera.xacro"/>
