Commit message: Update wheel configuration and odometry settings in Xacro files for improved simulation accuracy, to redue the drift

File: my_bot/description/gazebo_control.xacro (robot description, xacro)
@@ -6,6 +6,7 @@
             <left_joint>left_wheel_joint</left_joint>
             <right_joint>right_wheel_joint</right_joint>
-            <wheel_separation>0.23</wheel_separation>
-            <wheel_diameter>0.1</wheel_diameter>
+            <!-- Match the controller configuration -->
+            <wheel_separation>0.297</wheel_separation>
+            <wheel_diameter>0.066</wheel_diameter>
             <!-- Limits -->
             <max_wheel_torque>200.0</max_wheel_torque>
@@ -14,6 +15,8 @@
             <odometry_frame>odom</odometry_frame>
             <robot_base_frame>base_link</robot_base_frame>
-            <publish_odom>true</publish_odom>
-            <publish_odom_tf>true</publish_odom_tf>
+          <!-- Disable Gazebo-side odometry publication to avoid duplicate/conflicting odom/TF.
+              The controller should publish odometry/TF instead. -->
+          <publish_odom>true</publish_odom>
+          <publish_odom_tf>true</publish_odom_tf>
             <publish_wheel_tf>true</publish_wheel_tf>
         </plugin>

File: my_bot/description/robot_core.xacro (robot description, xacro)
@@ -2,5 +2,4 @@
 <robot xmlns:xacro="http://www.ros.org/wiki/xacro"  >
     <xacro:include filename="inertial_macros.xacro"/>
-    <!-- <xacro:property name="pi" value="3.14159265359"/> -->
     <material name="white">
         <color rgba="1 1 1 1"/>
@@ -20,4 +19,12 @@
     <!-- BASE LINK -->
     <link name="base_link">
+    </link>
+    <!-- BASE FOOTPRINT LINK -->
+    <joint name="base_footprint_joint" type="fixed">
+        <parent link="base_link"/>
+        <child link="base_footprint"/>
+        <origin xyz="0 0 0" rpy="0 0 0"/>
+    </joint>
+    <link name="base_footprint">
     </link>
     <!-- CHASSIS link -->
@@ -42,5 +49,5 @@
             <material name="orange"/>
         </collision>
-        <xacro:inertial_box mass="0.5" x="0.3" y="0.3" z="0.15">
+        <xacro:inertial_box mass="0.3" x="0.3" y="0.3" z="0.15">
             <origin xyz="0.15 0 0.075" rpy="0 0 0"/>
         </xacro:inertial_box>
@@ -59,5 +66,5 @@
         <visual>
             <geometry>
-                <cylinder length="0.02" radius="0.05"/>
+                <cylinder length="0.01" radius="0.05"/>
             </geometry>
             <material name="blue"/>
@@ -65,11 +72,11 @@
         <collision>
             <geometry>
-                <cylinder length="0.02" radius="0.05"/>
+                <sphere radius="0.05"/>
             </geometry>
             <material name="blue"/>
         </collision>
-        <xacro:inertial_cylinder mass="0.1" length="0.02" radius="0.05">
+        <xacro:inertial_sphere mass="0.1" radius="0.05">
             <origin xyz="0 0 0" rpy="0 0 0"/>
-        </xacro:inertial_cylinder>
+        </xacro:inertial_sphere>
     </link>
     <gazebo reference="left_wheel">
@@ -86,5 +93,5 @@
         <visual>
             <geometry>
-                <cylinder length="0.02" radius="0.05"/>
+                <cylinder length="0.01" radius="0.05"/>
             </geometry>
             <material name="blue"/>
@@ -92,11 +99,11 @@
         <collision>
             <geometry>
-                <cylinder length="0.02" radius="0.05"/>
+                <sphere radius="0.05"/>
             </geometry>
             <material name="blue"/>
         </collision>
-        <xacro:inertial_cylinder mass="0.1" length="0.02" radius="0.05">
+        <xacro:inertial_sphere mass="0.1" radius="0.05">
             <origin xyz="0 0 0" rpy="0 0 0"/>
-        </xacro:inertial_cylinder>
+        </xacro:inertial_sphere>
     </link>
     <gazebo reference="right_wheel">

File: my_bot/description/ros2_control.xacro (robot description, xacro)
@@ -36,6 +36,7 @@
             <left_joint>left_wheel_joint</left_joint>
             <right_joint>right_wheel_joint</right_joint>
-            <wheel_separation>0.23</wheel_separation>
-            <wheel_diameter>0.1</wheel_diameter>
+            <!-- Match the controller configuration: separation in meters, diameter = 2 * wheel_radius -->
+            <wheel_separation>0.297</wheel_separation>
+            <wheel_diameter>0.066</wheel_diameter>
             <!-- Limits -->
             <max_wheel_torque>200.0</max_wheel_torque>
@@ -44,6 +45,8 @@
             <odometry_frame>odom</odometry_frame>
             <robot_base_frame>base_link</robot_base_frame>
-            <publish_odom>true</publish_odom>
-            <publish_odom_tf>true</publish_odom_tf>
+          <!-- Disable Gazebo-side odometry publication to avoid duplicate/conflicting odom/TF.
+              Let the diff_drive_controller (ros2_control) publish odometry/TF. -->
+          <publish_odom>true</publish_odom>
+          <publish_odom_tf>true</publish_odom_tf>
             <publish_wheel_tf>true</publish_wheel_tf>
         </plugin>
