Commit message: Add Gazebo plugins, launch file, and obstacle world for simulation

File: my_bot/description/robot.urdf.xacro (robot description, xacro)
@@ -4,3 +4,4 @@
     <!-- <link name="base_link"></link> -->
     <xacro:include filename="robot_core.xacro"/>
+    <xacro:include filename="gazebo_plugins.xacro"/>
 </robot>

File: my_bot/description/robot_core.xacro (robot description, xacro)
@@ -43,4 +43,7 @@
         </xacro:inertial_box>
     </link>
+    <gazebo reference="chassis">
+        <material>Gazebo/Orange</material>
+    </gazebo>
     <!-- LEFT WHEEL LINK -->
     <joint name="left_wheel_joint" type="continuous">
@@ -67,4 +70,7 @@
         </xacro:inertial_cylinder>
     </link>
+    <gazebo reference="left_wheel">
+        <material>Gazebo/Blue </material>
+    </gazebo>
     <!-- RIGHT WHEEL LINK -->
     <joint name="right_wheel_joint" type="continuous">
@@ -91,4 +97,7 @@
         </xacro:inertial_cylinder>
     </link>
+    <gazebo reference="right_wheel">
+        <material>Gazebo/Blue </material>
+    </gazebo>
     <!-- CASTER WHEEL LINK -->
     <joint name="caster_wheel_joint" type="fixed">
@@ -114,3 +123,8 @@
         </xacro:inertial_sphere>
     </link>
+    <gazebo reference="caster_wheel">
+        <material>Gazebo/Black </material>
+        <mu1 value="0.0001"/>
+        <mu2 value="0.0001"/>
+    </gazebo>
 </robot>

Commit message: Refactor code structure for improved readability and maintainability and added the lidar and world

File: my_bot/description/robot.urdf.xacro (robot description, xacro)
@@ -5,3 +5,4 @@
     <xacro:include filename="robot_core.xacro"/>
     <xacro:include filename="gazebo_plugins.xacro"/>
+    <xacro:include filename="Lidar.xacro"/>
 </robot>

File: my_bot/description/robot_core.xacro (robot description, xacro)
@@ -8,4 +8,7 @@
     <material name="orange">
         <color rgba="1 0.3 0.1 1"/>
+    </material>
+    <material name="red">
+        <color rgba="1 0 0 1"/>
     </material>
     <material name="blue">

Commit message: Add VLP-16 sensor definition and integration into robot description

File: my_bot/description/robot.urdf.xacro (robot description, xacro)
@@ -14,5 +14,11 @@
     </xacro:unless>
     <!-- Sensors -->
+    <!-- changing -->
     <xacro:include filename="lidar.xacro"/>
+    <xacro:include filename="VLP-16.urdf.xacro"/>
+    <!-- Instantiate the VLP-16 sensor, connected to the chassis -->
+    <xacro:VLP-16 parent="chassis" name="velodyne_vlp16" topic="/velodyne_points" hz="10">
+        <origin xyz="0.1 0 0.195" rpy="0 0 0"/>
+    </xacro:VLP-16>
     <xacro:include filename="camera.xacro"/>
     <xacro:include filename="depth_camera.xacro"/>

Commit message: Update VLP-16 sensor position and add IMU sensor definition

File: my_bot/description/robot.urdf.xacro (robot description, xacro)
@@ -19,7 +19,16 @@
     <!-- Instantiate the VLP-16 sensor, connected to the chassis -->
     <xacro:VLP-16 parent="chassis" name="velodyne_vlp16" topic="/velodyne_points" hz="10">
-        <origin xyz="0.1 0 0.195" rpy="0 0 0"/>
+        <origin xyz="0.15 0 0.195" rpy="0 0 0"/>
     </xacro:VLP-16>
     <xacro:include filename="camera.xacro"/>
     <xacro:include filename="depth_camera.xacro"/>
+    <!-- IMU Sensor -->
+    <xacro:include filename="xsens_mti._imu.urdf.xacro"/>
+    <xacro:xsens_imu_mti
+        parent_link="chassis"
+        imu_name="imu_sensor"
+        topic_name="/imu/data"
+        xyz="0 0 0.15"
+        rpy="0 0 0"
+    />
 </robot>
