Commit message: updated

File: my_bot/description/lidar.xacro (robot description, xacro)
@@ -27,5 +27,5 @@
         <sensor name="laser" type="ray">
             <pose> 0 0 0 0 0 0</pose>
-            <visualize>true</visualize>
+            <visualize>false</visualize>
             <update_rate>10</update_rate>
             <ray>

File: my_bot/description/robot.urdf.xacro (robot description, xacro)
@@ -19,10 +19,10 @@
     <!-- Instantiate the VLP-16 sensor, connected to the chassis -->
     <xacro:VLP-16 parent="chassis" name="velodyne_vlp16" topic="/velodyne_points" hz="10">
-        <origin xyz="0.15 0 0.195" rpy="0 0 0"/>
+        <origin xyz="0.1 0 0.195" rpy="0 0 0"/>
     </xacro:VLP-16>
     <xacro:include filename="camera.xacro"/>
     <xacro:include filename="depth_camera.xacro"/>
     <!-- IMU Sensor -->
-    <xacro:include filename="xsens_mti._imu.urdf.xacro"/>
+    <!-- <xacro:include filename="xsens_mti._imu.urdf.xacro"/>
     <xacro:xsens_imu_mti
         parent_link="chassis"
@@ -31,4 +31,4 @@
         xyz="0 0 0.15"
         rpy="0 0 0"
-    />
+    /> -->
 </robot>

Commit message: feat: Upgrade robot to 4-wheel drive with 3D lidar and add 3D ramp world for navigation testing.

File: my_bot/description/lidar.xacro (robot description, xacro)
@@ -37,19 +37,22 @@
                         <max_angle>3.14</max_angle>
                     </horizontal>
+                    <vertical>
+                        <samples>16</samples>
+                        <resolution>1</resolution>
+                        <min_angle>-0.261799</min_angle>
+                        <max_angle>0.261799</max_angle>
+                    </vertical>
                 </scan>
                 <range>
                     <min>0.3</min>
                     <max>12</max>
-                    <resolution>0.3</resolution>
+                    <resolution>0.01</resolution>
                 </range>
             </ray>
             <plugin name="gazebo_ros_ray_sensor" filename="libgazebo_ros_ray_sensor.so">
-                <!-- <ros>
-                    <argument>~/out:=scan</argument>
-                </ros> -->
                 <ros>
-                    <remapping>~/out:=scan</remapping>
+                    <remapping>~/out:=/velodyne_points</remapping>
                 </ros>
-                <output_type>sensor_msgs/LaserScan</output_type>
+                <output_type>sensor_msgs/PointCloud2</output_type>
                 <frame_name>laser_frame</frame_name>
             </plugin>

File: my_bot/description/robot_core.xacro (robot description, xacro)
@@ -36,105 +36,62 @@
     <link name="chassis">
         <visual>
-            <origin xyz="0.15 0 0.075"/>
+            <origin xyz="0 0 0.075"/>
             <geometry>
-                <box size="0.3 0.3 0.15"/>
+                <box size="0.6 0.4 0.15"/>
             </geometry>
-            <material name="orange"/>
+            <material name="green">
+                <color rgba="0 1 0 1"/>
+            </material>
         </visual>
         <collision>
-            <origin xyz="0.15 0 0.075"/>
+            <origin xyz="0 0 0.075"/>
             <geometry>
-                <box size="0.3 0.3 0.15"/>
+                <box size="0.6 0.4 0.15"/>
             </geometry>
-            <material name="orange"/>
+            <material name="green"/>
         </collision>
-        <xacro:inertial_box mass="0.3" x="0.3" y="0.3" z="0.15">
-            <origin xyz="0.15 0 0.075" rpy="0 0 0"/>
+        <xacro:inertial_box mass="5.0" x="0.6" y="0.4" z="0.15">
+            <origin xyz="0 0 0.075" rpy="0 0 0"/>
         </xacro:inertial_box>
     </link>
     <gazebo reference="chassis">
-        <material>Gazebo/Orange</material>
+        <material>Gazebo/Green</material>
     </gazebo>
-    <!-- LEFT WHEEL LINK -->
-    <joint name="left_wheel_joint" type="continuous">
-        <parent link="base_link"/>
-        <child link="left_wheel"/>
-        <origin xyz="0 0.175 0" rpy="-${pi/2} 0 0"/>
-        <axis xyz="0 0 1"/>
-    </joint>
-    <link name="left_wheel">
-        <visual>
-            <geometry>
-                <cylinder length="0.01" radius="0.05"/>
-            </geometry>
-            <material name="blue"/>
-        </visual>
-        <collision>
-            <geometry>
-                <sphere radius="0.05"/>
-            </geometry>
-            <material name="blue"/>
-        </collision>
-        <xacro:inertial_sphere mass="0.1" radius="0.05">
-            <origin xyz="0 0 0" rpy="0 0 0"/>
-        </xacro:inertial_sphere>
-    </link>
-    <gazebo reference="left_wheel">
-        <material>Gazebo/Blue </material>
-    </gazebo>
-    <!-- RIGHT WHEEL LINK -->
-    <joint name="right_wheel_joint" type="continuous">
-        <parent link="base_link"/>
-        <child link="right_wheel"/>
-        <origin xyz="0 -0.175 0" rpy="${pi/2} 0 0"/>
-        <axis xyz="0 0 -1"/>
-    </joint>
-    <link name="right_wheel">
-        <visual>
-            <geometry>
-                <cylinder length="0.01" radius="0.05"/>
-            </geometry>
-            <material name="blue"/>
-        </visual>
-        <collision>
-            <geometry>
-                <sphere radius="0.05"/>
-            </geometry>
-            <material name="blue"/>
-        </collision>
-        <xacro:inertial_sphere mass="0.1" radius="0.05">
-            <origin xyz="0 0 0" rpy="0 0 0"/>
-        </xacro:inertial_sphere>
-    </link>
-    <gazebo reference="right_wheel">
-        <material>Gazebo/Blue </material>
-    </gazebo>
-    <!-- CASTER WHEEL LINK -->
-    <joint name="caster_wheel_joint" type="fixed">
-        <parent link="chassis"/>
-        <child link="caster_wheel"/>
-        <origin xyz="0.24 0 0"/>
-    </joint>
-    <link name="caster_wheel">
-        <visual>
-            <geometry>
-                <sphere radius="0.05"/>
-            </geometry>
-            <material name="black"/>
-        </visual>
-        <collision>
-            <geometry>
-                <sphere radius="0.05"/>
-            </geometry>
-            <material name="black"/>
-        </collision>
-        <xacro:inertial_sphere mass="0.1" radius="0.05">
-            <origin xyz="0 0 0" rpy="0 0 0"/>
-        </xacro:inertial_sphere>
-    </link>
-    <gazebo reference="caster_wheel">
-        <material>Gazebo/Black </material>
-        <mu1 value="0.0001"/>
-        <mu2 value="0.0001"/>
-    </gazebo>
+    <!-- WHEEL MACRO -->
+    <xacro:macro name="wheel_link" params="prefix offset_x offset_y">
+        <joint name="${prefix}_wheel_joint" type="continuous">
+            <parent link="base_link"/>
+            <child link="${prefix}_wheel"/>
+            <origin xyz="${offset_x} ${offset_y} 0" rpy="-${pi/2} 0 0"/>
+            <axis xyz="0 0 1"/>
+        </joint>
+        <link name="${prefix}_wheel">
+            <visual>
+                <geometry>
+                    <cylinder length="0.04" radius="0.1"/>
+                </geometry>
+                <material name="blue"/>
+            </visual>
+            <collision>
+                <geometry>
+                    <cylinder length="0.04" radius="0.1"/>
+                </geometry>
+                 <material name="blue"/>
+            </collision>
+            <xacro:inertial_sphere mass="0.5" radius="0.1">
+                <origin xyz="0 0 0" rpy="0 0 0"/>
+            </xacro:inertial_sphere>
+        </link>
+        <gazebo reference="${prefix}_wheel">
+            <material>Gazebo/Blue</material>
+            <mu1 value="2.0"/>
+            <mu2 value="2.0"/>
+        </gazebo>
+    </xacro:macro>
+    <!-- Create 4 Wheels -->
+    <xacro:wheel_link prefix="rear_left" offset_x="-0.2" offset_y="0.25"/>
+    <xacro:wheel_link prefix="rear_right" offset_x="-0.2" offset_y="-0.25"/>
+    <xacro:wheel_link prefix="front_left" offset_x="0.2" offset_y="0.25"/>
+    <xacro:wheel_link prefix="front_right" offset_x="0.2" offset_y="-0.25"/>
+    <!-- Remove Caster Wheel -->
 </robot>

File: my_bot/description/ros2_control.xacro (robot description, xacro)
@@ -5,16 +5,32 @@
             <plugin>gazebo_ros2_control/GazeboSystem</plugin>
         </hardware>
-        <joint name="left_wheel_joint">
+        <joint name="rear_left_wheel_joint">
             <command_interface name="velocity">
-                <param name="min">-10.0</param>
-                <param name="max">10.0</param>
+                <param name="min">-10</param>
+                <param name="max">10</param>
             </command_interface>
             <state_interface name="velocity"/>
             <state_interface name="position"/>
         </joint>
-        <joint name="right_wheel_joint">
+        <joint name="rear_right_wheel_joint">
             <command_interface name="velocity">
-                <param name="min">-10.0</param>
-                <param name="max">10.0</param>
+                <param name="min">-10</param>
+                <param name="max">10</param>
+            </command_interface>
+            <state_interface name="velocity"/>
+            <state_interface name="position"/>
+        </joint>
+        <joint name="front_left_wheel_joint">
+            <command_interface name="velocity">
+                <param name="min">-10</param>
+                <param name="max">10</param>
+            </command_interface>
+            <state_interface name="velocity"/>
+            <state_interface name="position"/>
+        </joint>
+        <joint name="front_right_wheel_joint">
+            <command_interface name="velocity">
+                <param name="min">-10</param>
+                <param name="max">10</param>
             </command_interface>
             <state_interface name="velocity"/>
