Commit message: changes wheel width, to reduce the drift

File: my_bot/description/robot_core.xacro (robot description, xacro)
@@ -59,5 +59,5 @@
         <visual>
             <geometry>
-                <cylinder length="0.04" radius="0.05"/>
+                <cylinder length="0.02" radius="0.05"/>
             </geometry>
             <material name="blue"/>
@@ -65,9 +65,9 @@
         <collision>
             <geometry>
-                <cylinder length="0.04" radius="0.05"/>
+                <cylinder length="0.02" radius="0.05"/>
             </geometry>
             <material name="blue"/>
         </collision>
-        <xacro:inertial_cylinder mass="0.1" length="0.04" radius="0.05">
+        <xacro:inertial_cylinder mass="0.1" length="0.02" radius="0.05">
             <origin xyz="0 0 0" rpy="0 0 0"/>
         </xacro:inertial_cylinder>
@@ -86,5 +86,5 @@
         <visual>
             <geometry>
-                <cylinder length="0.04" radius="0.05"/>
+                <cylinder length="0.02" radius="0.05"/>
             </geometry>
             <material name="blue"/>
@@ -92,9 +92,9 @@
         <collision>
             <geometry>
-                <cylinder length="0.04" radius="0.05"/>
+                <cylinder length="0.02" radius="0.05"/>
             </geometry>
             <material name="blue"/>
         </collision>
-        <xacro:inertial_cylinder mass="0.1" length="0.04" radius="0.05">
+        <xacro:inertial_cylinder mass="0.1" length="0.02" radius="0.05">
             <origin xyz="0 0 0" rpy="0 0 0"/>
         </xacro:inertial_cylinder>

Commit message: Convert robot to 2-wheel drive with casters, enhance 3D navigation with static Octomap support, and add a navigation test script.

File: my_bot/description/robot_core.xacro (robot description, xacro)
@@ -92,6 +92,59 @@
     <xacro:wheel_link prefix="rear_left" offset_x="-0.2" offset_y="0.25"/>
     <xacro:wheel_link prefix="rear_right" offset_x="-0.2" offset_y="-0.25"/>
-    <xacro:wheel_link prefix="front_left" offset_x="0.2" offset_y="0.25"/>
-    <xacro:wheel_link prefix="front_right" offset_x="0.2" offset_y="-0.25"/>
+    <!-- FRONT CASTER WHEELS (Passive, Low Friction) -->
+    <joint name="front_left_caster_joint" type="fixed">
+        <parent link="chassis"/>
+        <child link="front_left_caster"/>
+        <origin xyz="0.2 0.25 -0.05" rpy="0 0 0"/>
+    </joint>
+    <link name="front_left_caster">
+        <visual>
+            <geometry>
+                <sphere radius="0.05"/>
+            </geometry>
+            <material name="black"/>
+        </visual>
+        <collision>
+            <geometry>
+                <sphere radius="0.05"/>
+            </geometry>
+            <material name="black"/>
+        </collision>
+        <xacro:inertial_sphere mass="0.1" radius="0.05">
+            <origin xyz="0 0 0" rpy="0 0 0"/>
+        </xacro:inertial_sphere>
+    </link>
+    <gazebo reference="front_left_caster">
+        <material>Gazebo/Black</material>
+        <mu1 value="0.001"/>
+        <mu2 value="0.001"/>
+    </gazebo>
+    <joint name="front_right_caster_joint" type="fixed">
+        <parent link="chassis"/>
+        <child link="front_right_caster"/>
+        <origin xyz="0.2 -0.25 -0.05" rpy="0 0 0"/>
+    </joint>
+    <link name="front_right_caster">
+        <visual>
+            <geometry>
+                <sphere radius="0.05"/>
+            </geometry>
+            <material name="black"/>
+        </visual>
+        <collision>
+            <geometry>
+                <sphere radius="0.05"/>
+            </geometry>
+            <material name="black"/>
+        </collision>
+        <xacro:inertial_sphere mass="0.1" radius="0.05">
+            <origin xyz="0 0 0" rpy="0 0 0"/>
+        </xacro:inertial_sphere>
+    </link>
+    <gazebo reference="front_right_caster">
+        <material>Gazebo/Black</material>
+        <mu1 value="0.001"/>
+        <mu2 value="0.001"/>
+    </gazebo>
     <!-- Remove Caster Wheel -->
 </robot>

File: my_bot/description/ros2_control.xacro (robot description, xacro)
@@ -21,20 +21,5 @@
             <state_interface name="position"/>
         </joint>
-        <joint name="front_left_wheel_joint">
-            <command_interface name="velocity">
-                <param name="min">-10</param>
-                <param name="max">10</param>
-            </command_interface>
-            <state_interface name="velocity"/>
-            <state_interface name="position"/>
-        </joint>
-        <joint name="front_right_wheel_joint">
-            <command_interface name="velocity">
-                <param name="min">-10</param>
-                <param name="max">10</param>
-            </command_interface>
-            <state_interface name="velocity"/>
-            <state_interface name="position"/>
-        </joint>
+        <!-- FRONT WHEELS ARE PASSIVE CASTERS NOW -->
     </ros2_control>
     <gazebo>
